Commit message: worked on drone cad and sim

File: drone/drone.urdf (robot description, URDF)
Before this commit: robot drone, 1 links, 0 joints
Links:
- added link prop1; visual mesh filename=prop1.stl scale=0.001 0.001 0.001
- added link prop2; visual mesh filename=prop2.stl scale=0.001 0.001 0.001
- added link prop3; visual mesh filename=prop3.stl scale=0.001 0.001 0.001
- added link prop4; visual mesh filename=prop4.stl scale=0.001 0.001 0.001
Joints:
- added joint prop1_joint: type revolute, parent base, child prop1, origin xyz=-11.504 12.236 -0.289, axis 0 0 1, limit lower=-3.14 upper=3.14 effort=1 velocity=1000
- added joint prop2_joint: type revolute, parent base, child prop2, origin xyz=6.795 12.319 -0.441, axis 0 0 1, limit lower=-3.14 upper=3.14 effort=1 velocity=1000
- added joint prop3_joint: type revolute, parent base, child prop3, origin xyz=-10.643 -8.545 2.418, axis 0 0 1, limit lower=-3.14 upper=3.14 effort=1 velocity=1000
- added joint prop4_joint: type revolute, parent base, child prop4, origin xyz=6.527 -8.015 2.409, axis 0 0 1, limit lower=-3.14 upper=3.14 effort=1 velocity=1000

Commit message: idk

File: drone/drone.urdf (robot description, URDF)
Before this commit: robot drone, 5 links, 4 joints
Links:
- link prop1: mass None -> 0.01; geometry collision mesh filename=prop1.stl scale=0.001 0.001 0.001; visual mesh filename=prop1.stl scale=0.001 0.001 0.001
- link prop2: mass None -> 0.01; geometry collision mesh filename=prop2.stl scale=0.001 0.001 0.001; visual mesh filename=prop2.stl scale=0.001 0.001 0.001
- link prop3: mass None -> 0.01; geometry collision mesh filename=prop3.stl scale=0.001 0.001 0.001; visual mesh filename=prop3.stl scale=0.001 0.001 0.001
- link prop4: mass None -> 0.01; geometry collision mesh filename=prop4.stl scale=0.001 0.001 0.001; visual mesh filename=prop4.stl scale=0.001 0.001 0.001
Joints:
- joint prop1_joint: limit lower=-3.14 upper=3.14 effort=1 velocity=1000 -> (none); type revolute -> continuous
- joint prop2_joint: limit lower=-3.14 upper=3.14 effort=1 velocity=1000 -> (none); type revolute -> continuous
- joint prop3_joint: limit lower=-3.14 upper=3.14 effort=1 velocity=1000 -> (none); type revolute -> continuous
- joint prop4_joint: limit lower=-3.14 upper=3.14 effort=1 velocity=1000 -> (none); type revolute -> continuous
